Commit message: update so101-6dof urdf

File: sim/onshape_to_robot/so101_6dof/robot.urdf (robot description, URDF)
Before this commit: robot so101_6dof, 8 links, 7 joints
Links:
- removed link wrist_yaw_back_v1
- removed link wrist_yaw_front_v1
- added link wrist_yaw_back_v2, mass 1e-09; collision mesh filename=package://assets/wrist_yaw_back_v2.stl; visual mesh filename=package://assets/wrist_yaw_back_v2.stl
- added link wrist_yaw_front_v2, mass 0.11; collision mesh filename=package://assets/sts3215.stl; collision mesh filename=package://assets/sts3215.stl
Joints:
- removed joint joint 1
- removed joint joint 2
- removed joint joint 3
- removed joint joint 4
- removed joint joint 5
- removed joint joint 6
- removed joint joint 7
- added joint joint1: type revolute, parent base_so101_v2, child rotation_pitch_so101_v1, origin xyz=0.00025 -0.0449 0.0648 rpy=-3.14159 2.54451e-16 -1.5708, axis 0 0 1, limit lower=-1.91986 upper=1.91986 effort=10 velocity=10
- added joint joint2: type revolute, parent rotation_pitch_so101_v1, child upper_arm_so101_v1, origin xyz=0.0306 0.0183 -0.0542 rpy=1.5708 1.5708 0, axis 0 0 1, limit lower=-1.74534 upper=1.74532 effort=10 velocity=10
- added joint joint3: type revolute, parent upper_arm_so101_v1, child under_arm_so101_v1, origin xyz=0.11257 0.0280016 1.97758e-16 rpy=-6.19838e-16 -9.24429e-16 1.57081, axis 0 0 1, limit lower=-1.68946 upper=1.57081 effort=10 velocity=10
- added joint joint4: type revolute, parent under_arm_so101_v1, child wrist_yaw_back_v2, origin xyz=0.1349 -0.0052023 -4.57967e-16 rpy=2.15258e-14 -9.15934e-15 -1.70283e-05, axis 0 0 1, limit lower=-1.46608 upper=1.64061 effort=10 velocity=10
- added joint joint5: type revolute, parent wrist_yaw_back_v2, child wrist_yaw_front_v2, origin xyz=0.0290001 -0.0358999 0.0183 rpy=1.5708 -0.0151526 -3.14159, axis 0 0 1, limit lower=-1.55104 upper=1.52074 effort=10 velocity=10
- added joint joint6: type revolute, parent wrist_yaw_front_v2, child wrist_roll_follower_so101_v1, origin xyz=-0.0615 -8.67362e-19 0.037543 rpy=-3.14159 -1.5708 0, axis 0 0 1, limit lower=-2.96861 upper=2.86078 effort=10 velocity=10
- added joint joint7: type revolute, parent wrist_roll_follower_so101_v1, child moving_jaw_so101_v1, origin xyz=-0.020171 -0.0186314 -0.0234 rpy=1.5708 -5.80034e-15 -3.14004, axis 0 0 1, limit lower=-0.174533 upper=1.74533 effort=10 velocity=10
