Commit message: update so101_yaw urdf

File: sim/onshape_to_robot/so101_yaw/robot.urdf (robot description, URDF)
Before this commit: robot so101_yaw, 12 links, 11 joints
Links:
- removed link base_so101_v2
- removed link gripper_body
- removed link gripper_finger
- removed link moving_jaw_so101_v1
- removed link rotation_pitch_so101_v1
- removed link under_arm_so101_v1
- removed link upper_arm_so101_v1
- removed link wrist_yaw_back_v2
- removed link wrist_yaw_front_v2
- added link base, mass 0.151; collision mesh filename=package:///home/dhan/Desktop/study/d2lrobot/sim/onshape_to_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; collision mesh filename=package:///home/dhan/Desktop/study/d2lrobot/sim/onshape_to_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
- added link base_rotation, mass 0.102; collision mesh filename=package:///home/dhan/Desktop/study/d2lrobot/sim/onshape_to_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; collision mesh filename=package:///home/dhan/Desktop/study/d2lrobot/sim/onshape_to_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
- added link gripper_back, mass 1e-9
- added link gripper_center, mass 1e-9
- added link gripper_fixed, mass 0.086; collision mesh filename=package:///home/dhan/Desktop/study/d2lrobot/sim/onshape_to_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; collision mesh filename=package:///home/dhan/Desktop/study/d2lrobot/sim/onshape_to_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
- added link gripper_jaw, mass 0.013; collision mesh filename=package:///home/dhan/Desktop/study/d2lrobot/sim/onshape_to_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; collision mesh filename=package:///home/dhan/Desktop/study/d2lrobot/sim/onshape_to_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
- added link under_arm, mass 0.11; collision mesh filename=package:///home/dhan/Desktop/study/d2lrobot/sim/onshape_to_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; collision mesh filename=package:///home/dhan/Desktop/study/d2lrobot/sim/onshape_to_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
- added link upper_arm, mass 0.106; collision mesh filename=package:///home/dhan/Desktop/study/d2lrobot/sim/onshape_to_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; collision mesh filename=package:///home/dhan/Desktop/study/d2lrobot/sim/onshape_to_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
- added link wrist_yaw_back, mass 0.02; collision mesh filename=package:///home/dhan/Desktop/study/d2lrobot/sim/onshape_to_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; collision mesh filename=package:///home/dhan/Desktop/study/d2lrobot/sim/onshape_to_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
- added link wrist_yaw_front, mass 0.14; collision mesh filename=package:///home/dhan/Desktop/study/d2lrobot/sim/onshape_to_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; collision mesh filename=package:///home/dhan/Desktop/study/d2lrobot/sim/onshape_to_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
- link camera_body: geometry collision mesh filename=package:///home/dhan/Desktop/study/d2lrobot/sim/onshape_to_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; collision mesh filename=package:///home/dhan/Desktop/study/d2lrobot/sim/onshape_to_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
- link camera_mount: geometry collision mesh filename=package:///home/dhan/Desktop/study/d2lrobot/sim/onshape_to_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; collision mesh filename=package:///home/dhan/Desktop/study/d2lrobot/sim/onshape_to_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
Joints:
- removed joint joint8
- added joint gripper_back_frame: type fixed, parent gripper_fixed, child gripper_back, origin xyz=0 -0 -0.009 rpy=1.56714 1.5708 0, axis 0 0 0
- added joint gripper_center_frame: type fixed, parent gripper_fixed, child gripper_center, origin xyz=0 -0 -0.064 rpy=1.56714 1.5708 0, axis 0 0 0
- joint camera: limit effort=10 velocity=10 -> effort=3.3 velocity=5; origin xyz=-0.0299654 -0.0006 -0.0493488 rpy=3.14159 -0.436332 5.4113e-20 -> xyz=-0.0299654 -0.0006 -0.0493488 rpy=3.14159 -0.436332 0
- joint camera_frame: origin xyz=0.0134 0.000203456 -0.000397664 rpy=7.23838e-20 -2.65658e-17 1.24493e-19 -> xyz=0.0134 0.000203456 -0.000397664 rpy=-0 0 0
- joint camera_mount: limit effort=10 velocity=10 -> effort=3.3 velocity=5; origin xyz=-0.00306393 -0.0240046 -0.0234002 rpy=-1.5723 1.5708 0 -> xyz=-0.00301234 -0.0240112 -0.0234002 rpy=-1.57445 1.5708 0; parent gripper_body -> gripper_fixed
- joint joint1: child rotation_pitch_so101_v1 -> base_rotation; limit lower=-1.91986 upper=1.91986 effort=10 velocity=10 -> lower=-1.91986 upper=1.91986 effort=3.3 velocity=5; origin xyz=0.0173989 -0.0272511 0.0648 rpy=3.14159 -7.4744e-16 -3.26128e-15 -> xyz=0.0173989 -0.0272511 0.0648 rpy=3.14159 -0 -0; parent base_so101_v2 -> base
- joint joint2: child upper_arm_so101_v1 -> upper_arm; limit lower=-1.74533 upper=1.74533 effort=10 velocity=10 -> lower=-1.74533 upper=1.74533 effort=3.3 velocity=5; parent rotation_pitch_so101_v1 -> base_rotation
- joint joint3: child under_arm_so101_v1 -> under_arm; limit lower=-1.68948 upper=1.5708 effort=10 velocity=10 -> lower=-1.68948 upper=1.5708 effort=3.3 velocity=5; origin xyz=0.11257 0.028 -1.31839e-16 rpy=8.52564e-24 -1.11022e-16 1.5708 -> xyz=0.11257 0.028 -0 rpy=0 -0 1.5708; parent upper_arm_so101_v1 -> upper_arm
- joint joint4: child wrist_yaw_back_v2 -> wrist_yaw_back; limit lower=-1.46608 upper=1.64061 effort=10 velocity=10 -> lower=-1.46608 upper=1.64061 effort=3.3 velocity=5; origin xyz=0.1349 -0.0052 7.84095e-16 rpy=-1.01607e-15 1.38833e-15 -7.17499e-14 -> xyz=0.1349 -0.0052 -0 rpy=-0 0 -0; parent under_arm_so101_v1 -> under_arm
- joint joint5: child wrist_yaw_front_v2 -> wrist_yaw_front; limit lower=-1.53589 upper=1.53589 effort=10 velocity=10 -> lower=-1.54481 upper=1.52697 effort=3.3 velocity=5; origin xyz=0.029 -0.0359 0.0183 rpy=1.5708 4.20225e-14 -3.14159 -> xyz=0.029 -0.0359 0.0183 rpy=1.5708 -0.00891726 -3.14159; parent wrist_yaw_back_v2 -> wrist_yaw_back
- joint joint6: child gripper_body -> gripper_fixed; limit lower=-2.96856 upper=2.86084 effort=10 velocity=10 -> lower=-2.97071 upper=2.85869 effort=3.3 velocity=5; origin xyz=-0.0615 3.05311e-16 0.037543 rpy=-3.14159 -1.5708 0 -> xyz=-0.0615 0 0.037543 rpy=-3.14159 -1.5708 0; parent wrist_yaw_front_v2 -> wrist_yaw_front
- joint joint7: child moving_jaw_so101_v1 -> gripper_jaw; limit lower=-0.174109 upper=1.74575 effort=10 velocity=10 -> lower=-0.174123 upper=1.74574 effort=3.3 velocity=5; origin xyz=-0.020172 -0.0186303 -0.0234 rpy=1.5708 8.40848e-16 -3.14009 -> xyz=-0.0201319 -0.0186736 -0.0234 rpy=1.5708 0 -3.13794; parent gripper_body -> gripper_fixed
