Commit message: update urdf

File: sim/robot_urdf/so101_yaw/robot.urdf (robot description, URDF)
Before this commit: robot so101_yaw, 13 links, 12 joints
Links:
- link base: geometry collision box size=0.065 0.05 0.054; collision box size=0.1 0.11 0.02
- link base_rotation: geometry collision box size=0.037 0.054 0.03; collision box size=0.0554 0.0148 0.0396
- link camera_body: geometry visual mesh filename=package://assets/camera_uvc_25x32.stl
- link camera_mount: geometry visual mesh filename=package://assets/wrist_camera_mount.stl
- link gripper_fixed: geometry collision box size=0.02 0.033 0.04; collision box size=0.035 0.035 0.005
- link gripper_jaw: geometry collision mesh filename=package://assets/convex_decomposition/gripper_jaw_00006.stl; collision mesh filename=package://assets/convex_decomposition/gripper_jaw_00009.stl
- link under_arm: geometry collision box size=0.03 0.053 0.037; collision box size=0.092 0.062 0.025
- link upper_arm: geometry collision box size=0.062 0.028 0.052; collision box size=0.07 0.028 0.065
- link wrist_yaw_back: geometry collision cylinder length=0.045 radius=0.015; collision cylinder length=0.055 radius=0.012358
- link wrist_yaw_front: geometry collision box size=0.035 0.03 0.045; collision box size=0.05 0.033 0.04

File: sim/robot_urdf/so101_yaw_long/robot.urdf (robot description, URDF)
Before this commit: robot so101_yaw_long, 13 links, 12 joints
Links:
- link base: geometry collision box size=0.065 0.05 0.054; collision box size=0.1 0.11 0.02
- link base_rotation: geometry collision box size=0.037 0.054 0.03; collision box size=0.0754 0.0248 0.0396
- link camera_body: geometry visual mesh filename=package://assets/camera_uvc_25x32.stl
- link camera_mount: geometry visual mesh filename=package://assets/wrist_camera_mount.stl
- link gripper_fixed: geometry collision box size=0.02 0.033 0.04; collision box size=0.035 0.035 0.005
- link gripper_jaw: geometry collision mesh filename=package://assets/convex_decomposition/gripper_jaw_00006.stl; collision mesh filename=package://assets/convex_decomposition/gripper_jaw_00009.stl
- link under_arm: geometry collision box size=0.03 0.053 0.037; collision box size=0.15 0.062 0.025
- link upper_arm: geometry collision box size=0.08 0.028 0.065; collision box size=0.112 0.028 0.052
- link wrist_yaw_back: geometry collision cylinder length=0.045 radius=0.015; collision cylinder length=0.055 radius=0.012358
- link wrist_yaw_front: geometry collision box size=0.035 0.03 0.045; collision box size=0.05 0.033 0.04

File: sim/robot_urdf/xlerobot_yaw_long/xlerobot_yaw_long_armbase.urdf (robot description, URDF)
Before this commit: robot xlerobot_yaw_long, 24 links, 23 joints
Links:
- link armbase: geometry collision box size=0.05 0.06 0.055; collision box size=0.05 0.06 0.055
- link camera_mount1: geometry collision box size=0.02 0.06 0.06; visual mesh filename=package://assets/camera_mount1.stl
- link gimbal_yaw: geometry collision box size=0.045 0.032 0.047; visual mesh filename=package://assets/gimbal_yaw.stl
- link left_base_rotation: geometry collision box size=0.04 0.054 0.03; collision box size=0.0654 0.0148 0.0396
- link left_gripper_fixed: geometry collision box size=0.02 0.033 0.04; collision box size=0.035 0.035 0.005
- link left_gripper_jaw: geometry collision mesh filename=package://assets/convex_decomposition/gripper_jaw_00006.stl; collision mesh filename=package://assets/convex_decomposition/gripper_jaw_00009.stl
- link left_under_arm: geometry collision box size=0.03 0.055 0.033; collision box size=0.13 0.0615 0.025
- link left_upper_arm: geometry collision box size=0.08 0.03 0.065; collision box size=0.103 0.025 0.053
- link left_wrist_yaw_back: geometry collision cylinder length=0.045 radius=0.015; collision cylinder length=0.055 radius=0.012358
- link left_wrist_yaw_front: geometry collision box size=0.035 0.03 0.04; collision box size=0.05 0.033 0.04
- link right_base_rotation: geometry collision box size=0.04 0.054 0.03; collision box size=0.0554 0.015 0.04
- link right_gripper_fixed: geometry collision box size=0.02 0.033 0.04; collision box size=0.035 0.035 0.0055
- link right_gripper_jaw: geometry collision mesh filename=package://assets/convex_decomposition/gripper_jaw_2_00006.s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; collision mesh filename=package://assets/convex_decomposition/gripper_jaw_2_00009.s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
- link right_under_arm: geometry collision box size=0.03 0.055 0.033; collision box size=0.13 0.0615 0.025
- link right_upper_arm: geometry collision box size=0.08 0.03 0.065; collision box size=0.103 0.025 0.053
- link right_wrist_yaw_back: geometry collision cylinder length=0.045 radius=0.015; collision cylinder length=0.055 radius=0.012358
- link right_wrist_yaw_front: geometry collision box size=0.035 0.03 0.04; collision box size=0.05 0.033 0.04

File: sim/robot_urdf/xlerobot_yaw_long/xlerobot_yaw_long_full_back.urdf (robot description, URDF)
Before this commit: robot xlerobot_yaw_long, 28 links, 27 joints
Links:
- link armbase: geometry collision box size=0.05 0.06 0.055; collision box size=0.05 0.06 0.055
- link base: geometry collision box size=0.009 0.405 0.09; collision box size=0.009 0.405 0.09
- link camera_mount1: geometry collision box size=0.02 0.06 0.06; visual mesh filename=package://assets/camera_mount1.stl
- link gimbal_yaw: geometry collision box size=0.045 0.032 0.047; visual mesh filename=package://assets/gimbal_yaw.stl
- link left_base_rotation: geometry collision box size=0.04 0.054 0.03; collision box size=0.0654 0.0148 0.0396
- link left_gripper_fixed: geometry collision box size=0.02 0.033 0.04; collision box size=0.035 0.035 0.005
- link left_gripper_jaw: geometry collision mesh filename=package://assets/convex_decomposition/gripper_jaw_00006.stl; collision mesh filename=package://assets/convex_decomposition/gripper_jaw_00009.stl
- link left_under_arm: geometry collision box size=0.03 0.055 0.033; collision box size=0.13 0.0615 0.025
- link left_upper_arm: geometry collision box size=0.08 0.03 0.065; collision box size=0.103 0.025 0.053
- link left_wrist_yaw_back: geometry collision cylinder length=0.045 radius=0.015; collision cylinder length=0.055 radius=0.012358
- link left_wrist_yaw_front: geometry collision box size=0.035 0.03 0.04; collision box size=0.05 0.033 0.04
- link right_base_rotation: geometry collision box size=0.04 0.054 0.03; collision box size=0.0554 0.015 0.04
- link right_gripper_fixed: geometry collision box size=0.02 0.033 0.04; collision box size=0.035 0.035 0.0055
- link right_gripper_jaw: geometry collision mesh filename=package://assets/convex_decomposition/gripper_jaw_2_00006.s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; collision mesh filename=package://assets/convex_decomposition/gripper_jaw_2_00009.s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
- link right_under_arm: geometry collision box size=0.03 0.055 0.033; collision box size=0.13 0.0615 0.025
- link right_upper_arm: geometry collision box size=0.08 0.03 0.065; collision box size=0.103 0.025 0.053
- link right_wrist_yaw_back: geometry collision cylinder length=0.045 radius=0.015; collision cylinder length=0.055 radius=0.012358
- link right_wrist_yaw_front: geometry collision box size=0.035 0.03 0.04; collision box size=0.05 0.033 0.04

File: sim/robot_urdf/xlerobot_yaw_long/xlerobot_yaw_long_full_front.urdf (robot description, URDF)
Before this commit: robot xlerobot_yaw_long, 28 links, 27 joints
Links:
- link armbase: geometry collision box size=0.05 0.06 0.055; collision box size=0.05 0.06 0.055
- link base: geometry collision box size=0.009 0.405 0.09; collision box size=0.009 0.405 0.09
- link camera_mount1: geometry collision box size=0.02 0.06 0.06; visual mesh filename=package://assets/camera_mount1.stl
- link gimbal_yaw: geometry collision box size=0.045 0.032 0.047; visual mesh filename=package://assets/gimbal_yaw.stl
- link left_base_rotation: geometry collision box size=0.04 0.054 0.03; collision box size=0.0654 0.0148 0.0396
- link left_gripper_fixed: geometry collision box size=0.02 0.033 0.04; collision box size=0.035 0.035 0.005
- link left_gripper_jaw: geometry collision mesh filename=package://assets/convex_decomposition/gripper_jaw_00006.stl; collision mesh filename=package://assets/convex_decomposition/gripper_jaw_00009.stl
- link left_under_arm: geometry collision box size=0.03 0.055 0.033; collision box size=0.13 0.0615 0.025
- link left_upper_arm: geometry collision box size=0.08 0.03 0.065; collision box size=0.103 0.025 0.053
- link left_wrist_yaw_back: geometry collision cylinder length=0.045 radius=0.015; collision cylinder length=0.055 radius=0.012358
- link left_wrist_yaw_front: geometry collision box size=0.035 0.03 0.04; collision box size=0.05 0.033 0.04
- link right_base_rotation: geometry collision box size=0.04 0.054 0.03; collision box size=0.0554 0.015 0.04
- link right_gripper_fixed: geometry collision box size=0.02 0.033 0.04; collision box size=0.035 0.035 0.0055
- link right_gripper_jaw: geometry collision mesh filename=package://assets/convex_decomposition/gripper_jaw_2_00006.s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; collision mesh filename=package://assets/convex_decomposition/gripper_jaw_2_00009.s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
- link right_under_arm: geometry collision box size=0.03 0.055 0.033; collision box size=0.13 0.0615 0.025
- link right_upper_arm: geometry collision box size=0.08 0.03 0.065; collision box size=0.103 0.025 0.053
- link right_wrist_yaw_back: geometry collision cylinder length=0.045 radius=0.015; collision cylinder length=0.055 radius=0.012358
- link right_wrist_yaw_front: geometry collision box size=0.035 0.03 0.04; collision box size=0.05 0.033 0.04
